File: PCB/Kicad Files/Final PCB/Final PCB.kicad_pcb (KiCad board)
At the start: 2 copper layers, 189.5 x 148 mm, 54 parts, among them J1 Conn_01x20_Socket, J10 Conn_01x02_Socket, J11 Conn_01x02_Socket, J12 Conn_01x02_Socket, J13 Conn_01x02_Socket, J14 Conn_01x02_Socket, J15 Conn_01x02_Socket, J16 Conn_01x02_Socket, J17 Conn_01x02_Socket, J18 Conn_01x02_Socket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

Commit message: REFATORE: PCB altered with no CI 4049
Parts:
- removed J18, J19: Conn_01x02_Socket, Addlibrary:PinHeader_1x02_P2.54mm_VerticalLongPads
- removed R17, R18, R19, R20, R21, R22, R23, R24, R25, R26, R27, R28, R29, R30: R, Addlibrary:R_Axial_DIN0411_L9.9mm_D3.6mm_P25.40mm_HorizontalLongPads
- removed U1, U2, U3: 4049, Addlibrary:DIP-16_W7.62mm_Socket_LongPads
- added J2: Conn_01x02_Pin, Addlibrary:PinHeader_1x02_P2.54mm_VerticalLongPads, B.Cu at (89.0, 29.8)
- added J3: Conn_01x02_Pin, Addlibrary:PinHeader_1x02_P2.54mm_VerticalLongPads, B.Cu at (72.4, 29.8)
- added J4: Conn_01x02_Pin, Addlibrary:PinHeader_1x02_P2.54mm_VerticalLongPads, B.Cu at (138.9, 29.8)
- H1, H2, H3, H4: moved to B.Cu
- J10, J11, J12, J13, J14, J15, J16, J17, J5, J6, J7, J8, J9: value Conn_01x02_Socket -> Conn_01x02_Pin
- R1, R10, R11, R12, R13, R14, R15, R16, R2, R3, R4, R5, R6, R7, R8, R9: value R -> 100; footprint Addlibrary:R_Axial_DIN0411_L9.9mm_D3.6mm_P25.40mm_HorizontalLongPads -> Addlibrary:R_Axial_DIN0411_L9.9mm_D3.6mm_P12.70mm_HorizontalLONGPADS
- moved J14 138.0 mm to (155.6, 29.8), turned to 90 degrees
- moved R16 121.1 mm to (170.2, 120.7), turned to 90 degrees
- moved R13 120.3 mm to (155.6, 35.6)
- moved J10 112.0 mm to (146.0, 126.4), turned to 90 degrees
- moved J9 111.1 mm to (135.6, 126.4), turned to 90 degrees
- moved J11 109.1 mm to (94.0, 126.4), turned to 90 degrees
- moved J7 107.5 mm to (73.2, 126.4), turned to 90 degrees
- moved J8 107.1 mm to (83.6, 126.4), turned to 90 degrees
- moved R15 99.9 mm to (156.4, 120.7), turned to 90 degrees
- moved R3 90.1 mm to (138.9, 35.6)
- moved R4 80.9 mm to (122.3, 35.6)
- moved R2 79.5 mm to (72.4, 35.6)
- moved R1 78.9 mm to (89.0, 35.6)
- moved R5 78.3 mm to (105.7, 35.6)
- moved U6 75.9 mm to (113.0, 78.0)
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Connections:
- J1 pad 10: Net-(J1-Pin_10) -> /RR12
- J1 pad 11: Net-(J1-Pin_11) -> /RR4
- J1 pad 12: Net-(J1-Pin_12) -> /RR14
- J1 pad 13: Net-(J1-Pin_13) -> /RR5
- J1 pad 14: Net-(J1-Pin_14) -> /RR8
- J1 pad 15: Net-(J1-Pin_15) -> /RR1
- J1 pad 16: Net-(J1-Pin_16) -> /RR9
- J1 pad 17: Net-(J1-Pin_17) -> /RR2
- J1 pad 18: unconnected-(J1-Pin_18-Pad18) -> /RR15
- J1 pad 3: Net-(J1-Pin_3) -> /RR6
- J1 pad 4: Net-(J1-Pin_4) -> /RR7
- J1 pad 5: Net-(J1-Pin_5) -> unconnected-(J1-Pin_5-Pad5)
- J1 pad 6: Net-(J1-Pin_6) -> /RR10
- J1 pad 7: Net-(J1-Pin_7) -> /RR13
- J1 pad 8: Net-(J1-Pin_8) -> /RR11
- J1 pad 9: Net-(J1-Pin_9) -> /RR3
- J10 pad 2: Net-(J10-Pin_2) -> GND
- J11 pad 2: Net-(J11-Pin_2) -> GND
- J12 pad 2: Net-(J12-Pin_2) -> GND
- J13 pad 2: Net-(J13-Pin_2) -> GND
- J14 pad 2: Net-(J14-Pin_2) -> GND
- J15 pad 2: Net-(J15-Pin_2) -> GND
- J16 pad 2: Net-(J16-Pin_2) -> GND
- J17 pad 2: Net-(J17-Pin_2) -> GND
- J5 pad 2: Net-(J5-Pin_2) -> GND
- J6 pad 2: Net-(J6-Pin_2) -> GND
- J7 pad 2: Net-(J7-Pin_2) -> GND
- J8 pad 2: Net-(J8-Pin_2) -> GND
- J9 pad 2: Net-(J9-Pin_2) -> GND
- R1 pad 2: Net-(J14-Pin_1) -> /RR1
- R10 pad 1: Net-(J1-Pin_16) -> Net-(J11-Pin_1)
- R10 pad 2: Net-(J18-Pin_2) -> /RR10
- R11 pad 1: Net-(R11-Pad1) -> Net-(J12-Pin_1)
- R11 pad 2: Net-(J19-Pin_1) -> /RR11
- R12 pad 1: Net-(J1-Pin_17) -> Net-(J13-Pin_1)
- R12 pad 2: Net-(J19-Pin_2) -> /RR12
- R13 pad 1: Net-(R13-Pad1) -> Net-(J14-Pin_1)
- R13 pad 2: Net-(J13-Pin_1) -> /RR13
- R14 pad 1: Net-(J1-Pin_11) -> Net-(J15-Pin_1)
- R14 pad 2: Net-(J13-Pin_2) -> /RR14
- R15 pad 1: Net-(R15-Pad1) -> Net-(J16-Pin_1)
- R15 pad 2: Net-(J12-Pin_1) -> /RR15
- R16 pad 1: Net-(J1-Pin_10) -> Net-(J17-Pin_1)
- R16 pad 2: Net-(J12-Pin_2) -> /RR16
- R2 pad 1: Net-(J1-Pin_12) -> Net-(J3-Pin_1)
- R2 pad 2: Net-(J14-Pin_2) -> /RR2
- R3 pad 2: Net-(J15-Pin_1) -> /RR3
- R4 pad 1: Net-(J1-Pin_13) -> Net-(J5-Pin_1)
- R4 pad 2: Net-(J15-Pin_2) -> /RR4
- R5 pad 1: Net-(R5-Pad1) -> Net-(J6-Pin_1)
- R5 pad 2: Net-(J16-Pin_1) -> /RR5
- R6 pad 1: Net-(J1-Pin_14) -> Net-(J7-Pin_1)
- R6 pad 2: Net-(J16-Pin_2) -> /RR6
- R7 pad 1: Net-(R7-Pad1) -> Net-(J8-Pin_1)
- R7 pad 2: Net-(J17-Pin_1) -> /RR7
- R8 pad 1: Net-(J1-Pin_15) -> Net-(J9-Pin_1)
- R8 pad 2: Net-(J17-Pin_2) -> /RR8
- R9 pad 1: Net-(R9-Pad1) -> Net-(J10-Pin_1)
- R9 pad 2: Net-(J18-Pin_1) -> /RR9
- U6 pad 10: Net-(J1-Pin_12) -> /RR11
- U6 pad 11: Net-(J1-Pin_11) -> /RR10
- U6 pad 14: Net-(J1-Pin_10) -> /RR7
- U6 pad 15: Net-(J1-Pin_9) -> /RR6
- U6 pad 21: Net-(J1-Pin_8) -> /RR2
- U6 pad 22: Net-(J1-Pin_7) -> /RR1
- U6 pad 23: Net-(J1-Pin_6) -> /RR5
- U6 pad 24: Net-(J1-Pin_5) -> /RR4
- U6 pad 25: Net-(J1-Pin_4) -> /RR3
- U6 pad 26: Net-(J1-Pin_3) -> /RR13
- U6 pad 4: unconnected-(U6-D2-Pad4) -> /RR16
- U6 pad 5: Net-(J1-Pin_17) -> /RR15
- U6 pad 6: Net-(J1-Pin_16) -> /RR9
- U6 pad 7: Net-(J1-Pin_15) -> /RR8
- U6 pad 8: Net-(J1-Pin_14) -> /RR14
- U6 pad 9: Net-(J1-Pin_13) -> /RR12
Routing:
- net /RR15: track 0.00 -> 286.4 mm
- net /RR9: track 0.00 -> 279.1 mm
- net /RR8: track 0.00 -> 270.2 mm
- net +5V: track 0.00 -> 234.5 mm, vias 0 -> 2
- net Net-(J2-Pin_1): track 223.6 -> 5.72 mm
- net Net-(J4-Pin_1): track 190.0 -> 5.72 mm
- net /RR14: track 0.00 -> 171.7 mm
- net Net-(R5-Pad1): track 157.0 -> 0.00 mm
- net /RR12: track 0.00 -> 145.4 mm
- net /RR13: track 0.00 -> 131.2 mm
- net /RR11: track 0.00 -> 123.6 mm
- net /RR10: track 0.00 -> 112.1 mm
- net /RR3: track 0.00 -> 110.9 mm
- net /RR2: track 0.00 -> 108.6 mm
- net Net-(R7-Pad1): track 107.5 -> 0.00 mm
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- added copper zone on F.Cu, net GND
Other:
- board size 189.5 x 148 mm -> 165.1 x 120.6 mm
