File: PCB/Kicad V2/Principal PCB v2/Final PCB.kicad_pcb (KiCad board)
At the start: 2 copper layers, 165.1 x 120.6 mm, 38 parts, among them J1 Conn_01x20_Socket, J10 Conn_01x02_Pin, J11 Conn_01x02_Pin, J12 Conn_01x02_Pin, J13 Conn_01x02_Pin, J14 Conn_01x02_Pin, J15 Conn_01x02_Pin, J16 Conn_01x02_Pin, J17 Conn_01x02_Pin, J2 Conn_01x02_Pin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

Commit message: UPDATE final pcb finished and ADD secure backup module
Parts:
- added H10: MountingHole_Pad, Addlibrary:DefaultVia, B.Cu at (46.4, 97.8)
- added H5: MountingHole_Pad, Addlibrary:DefaultVia, B.Cu at (24.8, 97.8)
- added H6: MountingHole_Pad, Addlibrary:DefaultVia, B.Cu at (55.9, 106.0)
- added H7: MountingHole_Pad, Addlibrary:DefaultVia, B.Cu at (52.1, 47.6)
- added H8: MountingHole_Pad, Addlibrary:DefaultVia, B.Cu at (52.1, 60.3)
- added H9: MountingHole_Pad, Addlibrary:DefaultVia, B.Cu at (55.9, 121.9)
- moved H2 8.98 mm to (171.4, 31.8)
- moved H4 6.35 mm to (171.4, 133.3)
- moved H1 6.35 mm to (25.4, 31.8)
Routing:
- net +5V: track 234.5 -> 194.0 mm, vias 2 -> 0
- net /RR3: track 110.9 -> 113.5 mm
- net GND: track 39.0 -> 37.5 mm, vias 4 -> 0
- net /RR4: track 95.2 -> 96.6 mm
- net /RR8: track 270.2 -> 268.9 mm
- net /RR9: track 279.1 -> 277.8 mm
- net /RR15: track 286.4 -> 285.5 mm
- net /RR13: track 131.2 -> 131.9 mm
Other:
- board size 165.1 x 120.6 mm -> 158.8 x 114.3 mm
