File: PCB/Kicad V2/Principal PCB v2/Final PCB.kicad_sch (KiCad schematic)
At the start: 38 parts, among them J1 Conn_01x20_Socket, J10 Conn_01x02_Pin, J11 Conn_01x02_Pin, J12 Conn_01x02_Pin, J13 Conn_01x02_Pin, J14 Conn_01x02_Pin, J15 Conn_01x02_Pin, J16 Conn_01x02_Pin, J17 Conn_01x02_Pin, J2 Conn_01x02_Pin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

Commit message: UPDATE final pcb finished and ADD secure backup module
Parts:
- added H10, H5, H6, H7, H8, H9: MountingHole_Pad, Addlibrary:DefaultVia, symbol Mechanical:MountingHole_Pad
Connections:
- net +5V: now also H7.1, H8.1
- net GND: now also H10.1, H5.1, H6.1, H9.1
Other:
- company: (none) -> ETS - Robert Bosch Curitiba
- title: (none) -> Tool Manager PCB Schematic
- moved on the sheet: H1, H2, H3, H4, J1
